File: electrical/pcb/network-drone-fc/network-drone-fc.kicad_sch (KiCad schematic)
At the start: 79 parts, among them J1 U.FL-R-SMT-1, J2 TYPE-C 16PIN 2MD, J3 U.FL GPS, J4 ESC, J5 I2C port, J7 Charging board, U1 ESP32-S3FN8, U2 USBLC6-2SC6, U3 AP63205WU-7, U4 TLV75733PDRVR, U5 TPS7A2033PDBVR, U6 ICM-42688-P, U7 BMP581, U8 MAX-M10S, X1 Q22FA12800101

Commit message: Schematic: J5 becomes a 5 V sensor port (TF-Luna); J6 radio port added (5 V UART for the VoCore2)
J6 TX and RX share GPIO2 and GPIO10 with J4 pins 3 and 4. ERC 0 errors, 0 warnings.
Parts:
- added J6: Radio UART 5V, tar_fc:JST_SH_BM04B-SRSS-TB_1x04_Vertical, symbol tar_fc:SM04B-GHS-TB
- J5: value I2C port -> Sensor port 5V I2C
Connections:
- net +3V3: no longer J5.1
- net +5V: now also J5.1, J6.1
- net ESC_CUR: now also J6.2
- net ESC_TELEM: now also J6.3
- net GND: now also J6.4, J6.5, J6.6
Other:
- note added: "Sensor port J5 (TF-Luna): 5V, SCL, SDA, GND. Charging port J7: GND, DOCK_DET, AUX_ADC, spare. Radio port J6: 5V, TX (GPIO2), RX (GPIO10), GND. It shares the ESC CUR and TLM pins: use the ESC signals or the radio, not both."
- note removed: "I2C port uses the Dronecode order: VCC, SCL, SDA, GND. Charging port: GND, DOCK_DET, AUX_ADC, spare."
